Commit message: ros2_control for gazebo added

File: scara_description/urdf/scara.urdf.xacro (robot description, xacro)
@@ -4,3 +4,5 @@
     <xacro:include filename="materials.xacro" />
     <xacro:include filename="scara_core.xacro" />
+    <xacro:include filename="scara.ros2_control.xacro" />
+    <xacro:include filename="gz_plugins.xacro" />
 </robot>

File: scara_description/urdf/scara_core.xacro (robot description, xacro)
@@ -5,5 +5,5 @@
     <xacro:property name="base_ly" value="0.5" />
     <xacro:property name="base_lz" value="0.2" />
-    <xacro:property name="base_mass" value="2" />
+    <xacro:property name="base_mass" value="16" />
     <xacro:property name="column1_lx" value="0.2" />
     <xacro:property name="column1_ly" value="0.3" />
@@ -46,5 +46,5 @@
         <parent link="base_footprint" />
         <child link="base_link" />
-        <origin xyz="0 0.0 0.0" rpy="0.0 0.0 0.0" />
+        <origin xyz="0 0 ${base_lz / 2}" rpy="0.0 0.0 0.0" />
     </joint>
     <!-- Column 1 link -->
