Commit message: moving robotic arm from ros2 node

File: scara_description/urdf/scara_core.xacro (robot description, xacro)
@@ -4,5 +4,5 @@
     <xacro:property name="base_lx" value="0.5" />
     <xacro:property name="base_ly" value="0.5" />
-    <xacro:property name="base_lz" value="0.2" />
+    <xacro:property name="base_lz" value="0.35" />
     <xacro:property name="base_mass" value="16" />
     <xacro:property name="column1_lx" value="0.2" />

Commit message: added camera joint

File: scara_description/urdf/scara_core.xacro (robot description, xacro)
@@ -25,4 +25,7 @@
     <xacro:property name="ef_len" value="0.1" />
     <xacro:property name="ef_mass" value="0.1" />
+    <xacro:property name="camera_lx" value="0.02" />
+    <xacro:property name="camera_ly" value="0.02" />
+    <xacro:property name="camera_lz" value="0.02" />
     <!-- Base -->
     <link name="base_footprint" />
@@ -164,3 +167,17 @@
         <child link="ef_link" />
     </joint>
+    <link name="camera_link">
+        <visual>
+            <origin xyz="${camera_lx / 2} 0 0" rpy="0 0 0"/>
+            <geometry>
+                <box size="${camera_lx} ${camera_ly} ${camera_lz}"/>
+            </geometry>
+            <material name="black" />
+        </visual>
+    </link>
+    <joint name="elbow_camera_joint" type="fixed">
+        <origin xyz="${elbow_lx} 0 0" rpy="0 ${pi/2} 0"/>
+        <parent link="elbow_link"/>
+        <child link="camera_link"/>
+    </joint>
 </robot>
