Commit message: camera in tongue (boring name: coaxial vision system)

File: scara_description/urdf/gz_plugins.xacro (robot description, xacro)
@@ -21,5 +21,5 @@
     </gazebo>
     <gazebo reference="camera_link">
-        <sensor name="elbow_camera" type="camera">
+        <sensor name="ef_camera" type="camera">
             <always_on>true</always_on>
             <update_rate>30</update_rate>

File: scara_description/urdf/scara_core.xacro (robot description, xacro)
@@ -169,5 +169,5 @@
     <link name="camera_link">
         <visual>
-            <origin xyz="${camera_lx / 2} 0 0" rpy="0 0 0"/>
+            <origin xyz="0 0 0" rpy="0 0 0"/>
             <geometry>
                 <box size="${camera_lx} ${camera_ly} ${camera_lz}"/>
@@ -176,7 +176,7 @@
         </visual>
     </link>
-    <joint name="elbow_camera_joint" type="fixed">
-        <origin xyz="${elbow_lx} 0 0" rpy="0 ${pi/2} 0"/>
-        <parent link="elbow_link"/>
+    <joint name="ef_camera_joint" type="fixed">
+        <origin xyz="0 0 0" rpy="0 ${pi/2} 0"/>
+        <parent link="ef_link"/>
         <child link="camera_link"/>
     </joint>
