Commit message: fixed z stage physical movement issue

File: litho_ws/src/stage_description/urdf/inertials.xacro (robot description, xacro)
@@ -6,5 +6,5 @@
             <mass value="${m}" />
             <inertia ixx="${m/12 * (ly**2 + lz**2)}" ixy="0.0" ixz="0.0"
-                iyy="${m/12 * (lx**2 + lz**2)}" iyz="0.0" izz="${m/12 * (lx**2 + lz**2)}" />
+                iyy="${m/12 * (lx**2 + lz**2)}" iyz="0.0" izz="${m/12 * (lx**2 + ly**2)}" />
         </inertial>
     </xacro:macro>

File: litho_ws/src/stage_description/urdf/stage_core.xacro (robot description, xacro)
@@ -21,8 +21,8 @@
     <xacro:property name="z_stage_lz" value="0.01" />
     <xacro:property name="z_stage_mass" value="0.05" />
-    <xacro:property name="z_stage_lower" value="0" />
+    <xacro:property name="z_stage_lower" value="-0.025" />
     <xacro:property name="z_stage_upper" value="0.025" />
     <xacro:property name="stage_effort" value="100" /> <!-- N/m -->
-    <xacro:property name="stage_vel" value="0.005" /> <!-- m/s -->
+    <xacro:property name="stage_vel" value="0.1" /> <!-- m/s -->
     <!-- Base -->
     <link name="base_footprint" />
