Commit message: added camera

File: litho_ws/src/stage_description/urdf/gz_plugins.xacro (robot description, xacro)
@@ -1,4 +1,10 @@
 <?xml version="1.0"?>
 <robot xmlns:xacro="http://www.ros.org/wiki/xacro">
+    <gazebo>
+        <plugin filename="gz-sim-sensors-system"
+            name="gz::sim::systems::Sensors">
+            <render_engine>ogre2</render_engine>
+        </plugin>
+    </gazebo>
     <gazebo>
         <plugin filename="gz_ros2_control-system" name="gz_ros2_control::GazeboSimROS2ControlPlugin">
@@ -6,3 +12,31 @@
         </plugin>
     </gazebo>
+    <gazebo reference="camera_link">
+        <sensor name="camera" type="camera">
+            <camera>
+                <!-- <horizontal_fov>0.1</horizontal_fov> -->
+                <horizontal_fov>3.14</horizontal_fov>
+                <image>
+                    <width>640</width>
+                    <height>480</height>
+                    <format>R8G8B8</format>
+                </image>
+                <clip>
+                    <near>0.1</near>
+                    <far>0.2</far>
+                </clip>
+                <!-- <noise>
+                    <type>gaussian</type>
+                    <mean>0.0</mean>
+                    <stddev>0.007</stddev>
+                </noise> -->
+                <optical_frame_id>camera_link_optical</optical_frame_id>
+                <camera_info_topic>camera/camera_info</camera_info_topic>
+            </camera>
+            <always_on>1</always_on>
+            <update_rate>20</update_rate>
+            <visualize>true</visualize>
+            <topic>camera/image</topic>
+        </sensor>
+    </gazebo>
 </robot>

File: litho_ws/src/stage_description/urdf/stage_core.xacro (robot description, xacro)
@@ -14,5 +14,5 @@
     <xacro:property name="x_stage_lz" value="0.015" />
     <xacro:property name="x_stage_mass" value="0.1" />
-    <xacro:property name="x_stage_lower" value="0" />
+    <xacro:property name="x_stage_lower" value="-0.025" />
     <xacro:property name="x_stage_upper" value="0.025" />
     <xacro:property name="y_stage_lx" value="0.15" />
@@ -20,5 +20,5 @@
     <xacro:property name="y_stage_lz" value="0.015" />
     <xacro:property name="y_stage_mass" value="0.1" />
-    <xacro:property name="y_stage_lower" value="0" />
+    <xacro:property name="y_stage_lower" value="-0.025" />
     <xacro:property name="y_stage_upper" value="0.025" />
     <xacro:property name="z_stage_lx" value="0.1" />
@@ -34,5 +34,5 @@
     <link name="base_link">
         <visual>
-            <origin xyz="0 ${base_lz/2} 0" rpy="0 0 0" />
+            <origin xyz="0 0 ${base_lz/2}" rpy="0 0 0" />
             <geometry>
                 <box size="${base_lx} ${base_ly} ${base_lz}" />
@@ -41,5 +41,5 @@
         </visual>
         <collision>
-            <origin xyz="0 ${base_lz/2} 0" rpy="0 0 0" />
+            <origin xyz="0 0 ${base_lz/2}" rpy="0 0 0" />
             <geometry>
                 <box size="${base_lx} ${base_ly} ${base_lz}" />
@@ -47,5 +47,5 @@
         </collision>
         <xacro:box_inertial lx="${base_lx}" ly="${base_ly}" lz="${base_lz}" m="${base_mass}"
-            o_xyz="0 ${base_lz/2} 0" o_rpy="0 0 0" />
+            o_xyz="0 0 ${base_lz/2}" o_rpy="0 0 0" />
     </link>
     <joint name="footprint_base_joint" type="fixed">
@@ -152,5 +152,5 @@
     </link>
     <joint name="y_z_stage_joint" type="prismatic">
-        <origin xyz="0 0 ${y_stage_lz}" rpy="0 0 0" />
+        <origin xyz="0 0 ${y_stage_lz  + -z_stage_lower}" rpy="0 0 0" />
         <parent link="y_stage_link" />
         <child link="z_stage_link" />

Commit message: added bad wafer model

File: litho_ws/src/stage_description/urdf/gz_plugins.xacro (robot description, xacro)
@@ -15,8 +15,8 @@
         <sensor name="camera" type="camera">
             <camera>
-                <horizontal_fov>0.1</horizontal_fov>
+                <horizontal_fov>0.25</horizontal_fov> <!-- 0.25 or 0.1-->
                 <image>
-                    <width>640</width>
-                    <height>480</height>
+                    <width>800</width>  <!-- was 640 or 800 -->
+                    <height>600</height> <!-- was 480 or 600 -->
                     <format>R8G8B8</format>
                 </image>

File: litho_ws/src/stage_description/urdf/stage_core.xacro (robot description, xacro)
@@ -9,23 +9,23 @@
     <xacro:property name="camera_lz" value="0.01" />
     <xacro:property name="camera_mass" value="0.05" />
-    <xacro:property name="camera_offset_z" value="0.05" />
+    <xacro:property name="camera_offset_z" value="0.1" />
     <xacro:property name="x_stage_lx" value="0.15" />
     <xacro:property name="x_stage_ly" value="0.15" />
     <xacro:property name="x_stage_lz" value="0.015" />
     <xacro:property name="x_stage_mass" value="0.1" />
-    <xacro:property name="x_stage_lower" value="-0.025" />
-    <xacro:property name="x_stage_upper" value="0.025" />
+    <xacro:property name="x_stage_lower" value="-0.05" />
+    <xacro:property name="x_stage_upper" value="0.05" />
     <xacro:property name="y_stage_lx" value="0.15" />
     <xacro:property name="y_stage_ly" value="0.15" />
     <xacro:property name="y_stage_lz" value="0.015" />
     <xacro:property name="y_stage_mass" value="0.1" />
-    <xacro:property name="y_stage_lower" value="-0.025" />
-    <xacro:property name="y_stage_upper" value="0.025" />
+    <xacro:property name="y_stage_lower" value="-0.05" />
+    <xacro:property name="y_stage_upper" value="0.05" />
     <xacro:property name="z_stage_lx" value="0.1" />
     <xacro:property name="z_stage_ly" value="0.1" />
     <xacro:property name="z_stage_lz" value="0.01" />
     <xacro:property name="z_stage_mass" value="0.05" />
-    <xacro:property name="z_stage_lower" value="-0.025" />
-    <xacro:property name="z_stage_upper" value="0.025" />
+    <xacro:property name="z_stage_lower" value="-0.05" />
+    <xacro:property name="z_stage_upper" value="0.05" />
     <xacro:property name="stage_effort" value="100" /> <!-- N/m -->
     <xacro:property name="stage_vel" value="0.1" /> <!-- m/s -->
