Commit message: updated .gitignore, fixed stage wrong joint positioning

File: litho_ws/src/stage_description/urdf/stage_core.xacro (robot description, xacro)
@@ -13,9 +13,17 @@
     <xacro:property name="z_stage_ly" value="0.1" />
     <xacro:property name="z_stage_lz" value="0.01" />
+    <xacro:property name="x_stage_lower" value="0" />
+    <xacro:property name="x_stage_upper" value="0.025" />
+    <xacro:property name="y_stage_lower" value="0" />
+    <xacro:property name="y_stage_upper" value="0.025" />
+    <xacro:property name="z_stage_lower" value="0" />
+    <xacro:property name="z_stage_upper" value="0.025" />
+    <xacro:property name="stage_effort" value="100" />
+    <xacro:property name="stage_vel" value="0.0001" />
     <!-- Base -->
     <link name="base_footprint" />
     <link name="base_link">
         <visual>
-            <origin xyz="0 0 0" rpy="0 0 0" />
+            <origin xyz="0 ${base_lz/2} 0" rpy="0 0 0" />
             <geometry>
                 <box size="${base_lx} ${base_ly} ${base_lz}" />
@@ -25,5 +33,5 @@
     </link>
     <joint name="footprint_base_joint" type="fixed">
-        <origin xyz="0 0 ${base_lz / 2}" rpy="0 0 0" />
+        <origin xyz="0 0 ${base_lz/2}" rpy="0 0 0" />
         <parent link="base_footprint" />
         <child link="base_link" />
@@ -32,5 +40,5 @@
     <link name="x_stage_link">
         <visual>
-            <origin xyz="0 0 0" rpy="0 0 0" />
+            <origin xyz="0 0 ${x_stage_lz/2}" rpy="0 0 0" />
             <geometry>
                 <box size="${x_stage_lx} ${x_stage_ly} ${x_stage_lz}" />
@@ -40,14 +48,15 @@
     </link>
     <joint name="base_x_stage_joint" type="prismatic">
-        <origin xyz="0 0 ${x_stage_lz / 2}" rpy="0 0 0" />
+        <origin xyz="0 0 ${base_lz/2}" rpy="0 0 0" />
         <parent link="base_link" />
         <child link="x_stage_link" />
         <axis xyz="1 0 0" />
-        <limit lower="0.0" upper="0.025" effort="100" velocity="0.1" />
+        <limit lower="${x_stage_lower}" upper="${x_stage_upper}" effort="${stage_effort}"
+            velocity="${stage_vel}" />
     </joint>
     <!-- Y Stage -->
     <link name="y_stage_link">
         <visual>
-            <origin xyz="0 0 0" rpy="0 0 0" />
+            <origin xyz="0 0 ${y_stage_lz/2}" rpy="0 0 0" />
             <geometry>
                 <box size="${y_stage_lx} ${y_stage_ly} ${y_stage_lz}" />
@@ -57,14 +66,15 @@
     </link>
     <joint name="x_y_stage_joint" type="prismatic">
-        <origin xyz="0 0 ${y_stage_lz / 2}" rpy="0 0 0" />
+        <origin xyz="0 0 ${x_stage_lz}" rpy="0 0 0" />
         <parent link="x_stage_link" />
         <child link="y_stage_link" />
         <axis xyz="0 1 0" />
-        <limit lower="0.0" upper="0.025" effort="100" velocity="0.1" />
+        <limit lower="${y_stage_lower}" upper="${y_stage_upper}" effort="${stage_effort}"
+            velocity="${stage_vel}" />
     </joint>
     <!-- Z Stage -->
     <link name="z_stage_link">
         <visual>
-            <origin xyz="0 0 0" rpy="0 0 0" />
+            <origin xyz="0 0 ${z_stage_lz/2}" rpy="0 0 0" />
             <geometry>
                 <box size="${z_stage_lx} ${z_stage_ly} ${z_stage_lz}" />
@@ -74,9 +84,10 @@
     </link>
     <joint name="y_z_stage_joint" type="prismatic">
-        <origin xyz="0 0 ${z_stage_lz / 2}" rpy="0 0 0" />
+        <origin xyz="0 0 ${y_stage_lz}" rpy="0 0 0" />
         <parent link="y_stage_link" />
         <child link="z_stage_link" />
         <axis xyz="0 0 1" />
-        <limit lower="0.0" upper="0.025" effort="100" velocity="0.1" />
+        <limit lower="${z_stage_lower}" upper="${z_stage_upper}" effort="${stage_effort}"
+            velocity="${stage_vel}" />
     </joint>
 </robot>

Commit message: added camera link

File: litho_ws/src/stage_description/urdf/stage_core.xacro (robot description, xacro)
@@ -5,4 +5,9 @@
     <xacro:property name="base_lz" value="0.02" />
     <xacro:property name="base_mass" value="10" />
+    <xacro:property name="camera_lx" value="0.03" />
+    <xacro:property name="camera_ly" value="0.01" />
+    <xacro:property name="camera_lz" value="0.01" />
+    <xacro:property name="camera_mass" value="0.05" />
+    <xacro:property name="camera_offset_z" value="0.05" />
     <xacro:property name="x_stage_lx" value="0.15" />
     <xacro:property name="x_stage_ly" value="0.15" />
@@ -48,4 +53,28 @@
         <parent link="base_footprint" />
         <child link="base_link" />
+    </joint>
+    <!-- Camera -->
+    <link name="camera_link">
+        <visual>
+            <origin xyz="-${camera_lx/2} 0 0" rpy="0 0 0" />
+            <geometry>
+                <box size="${camera_lx} ${camera_ly} ${camera_lz}" />
+            </geometry>
+            <material name="reddishgrey" />
+        </visual>
+        <collision>
+            <origin xyz="-${camera_lx/2} 0 0" rpy="0 0 0" />
+            <geometry>
+                <box size="${camera_lx} ${camera_ly} ${camera_lz}" />
+            </geometry>
+        </collision>
+        <xacro:box_inertial lx="${camera_lx}" ly="${camera_ly}" lz="${camera_lz}" m="${camera_mass}"
+            o_xyz="-${camera_lx/2} 0 0" o_rpy="0 0 0" />
+    </link>
+    <joint name="base_camera_joint" type="fixed">
+        <origin xyz="0 0 ${base_lz/2 + x_stage_lz + y_stage_lz + z_stage_lz + camera_offset_z}"
+            rpy="0 ${pi/2} 0" />
+        <parent link="base_link" />
+        <child link="camera_link" />
     </joint>
     <!-- X Stage -->

Commit message: improved autoa lignment

File: litho_ws/src/stage_description/urdf/stage_core.xacro (robot description, xacro)
@@ -28,5 +28,6 @@
     <xacro:property name="z_stage_lower" value="-0.05" />
     <xacro:property name="z_stage_upper" value="0.05" />
-    <xacro:property name="stage_effort" value="100" /> <!-- N/m -->
+    <xacro:property name="z_stage_safety_lim" value="0.005" />
+    <xacro:property name="stage_effort" value="9999999999999999" /> <!-- N/m -->
     <xacro:property name="stage_vel" value="0.1" /> <!-- m/s -->
     <!-- Base -->
@@ -156,5 +157,5 @@
         <child link="z_stage_link" />
         <axis xyz="0 0 1" />
-        <limit lower="${z_stage_lower}" upper="${z_stage_upper}" effort="${stage_effort}"
+        <limit lower="${z_stage_lower + z_stage_safety_lim}" upper="${z_stage_upper - z_stage_safety_lim}" effort="${stage_effort}"
             velocity="${stage_vel}" />
     </joint>
